Commit message: Adds RViz Visualization for Go2
- Updated README.md for RViz use
- Changed feet step size in RLLocomotionContactController from 0.2 to 0.1 meters for better control.
- Removed deprecated state_publisher.py and several unused contact policy files.
- Introduced new launch files for go2 visualization in RViz and updated URDF paths for better compatibility.

File: src/robots/go2/go2_description/urdf/go2_description.urdf (robot description, URDF)
Before this commit: robot go2_description, 42 links, 41 joints
Links:
- removed link FL_calf_rotor
- removed link FL_hip_rotor
- removed link FL_thigh_rotor
- removed link FR_calf_rotor
- removed link FR_hip_rotor
- removed link FR_thigh_rotor
- removed link RL_calf_rotor
- removed link RL_hip_rotor
- removed link RL_thigh_rotor
- removed link RR_calf_rotor
- removed link RR_hip_rotor
- removed link RR_thigh_rotor
- removed link base
- removed link front_camera
- added link base_link, mass 6.921; collision box size=0.3762 0.0935 0.114; visual mesh filename=package://go2_description/dae/base.dae
- link FL_calf: geometry collision cylinder length=0.12 radius=0.012; visual mesh filename=package://go2_description/dae/calf.dae
- link FL_foot: geometry collision sphere radius=0.022; visual mesh filename=package://go2_description/dae/foot.dae
- link FL_hip: geometry collision cylinder length=0.04 radius=0.046; visual mesh filename=package://go2_description/dae/hip.dae
- link FL_thigh: geometry collision box size=0.213 0.0245 0.034; visual mesh filename=package://go2_description/dae/thigh.dae
- link FR_calf: geometry collision cylinder length=0.12 radius=0.013; visual mesh filename=package://go2_description/dae/calf_mirror.dae
- link FR_foot: geometry collision sphere radius=0.022; visual mesh filename=package://go2_description/dae/foot.dae
- link FR_hip: geometry collision cylinder length=0.04 radius=0.046; visual mesh filename=package://go2_description/dae/hip.dae
- link FR_thigh: geometry collision box size=0.213 0.0245 0.034; visual mesh filename=package://go2_description/dae/thigh_mirror.dae
- link RL_calf: geometry collision cylinder length=0.12 radius=0.013; visual mesh filename=package://go2_description/dae/calf.dae
- link RL_foot: geometry collision sphere radius=0.022; visual mesh filename=package://go2_description/dae/foot.dae
- link RL_hip: geometry collision cylinder length=0.04 radius=0.046; visual mesh filename=package://go2_description/dae/hip.dae
- link RL_thigh: geometry collision box size=0.213 0.0245 0.034; visual mesh filename=package://go2_description/dae/thigh.dae
- link RR_calf: geometry collision cylinder length=0.12 radius=0.013; visual mesh filename=package://go2_description/dae/calf_mirror.dae
- link RR_foot: geometry collision sphere radius=0.022; visual mesh filename=package://go2_description/dae/foot.dae
- link RR_hip: geometry collision cylinder length=0.04 radius=0.046; visual mesh filename=package://go2_description/dae/hip.dae
- link RR_thigh: geometry collision box size=0.213 0.0245 0.034; visual mesh filename=package://go2_description/dae/thigh_mirror.dae
Joints:
- removed joint FL_calf_rotor_joint
- removed joint FL_hip_rotor_joint
- removed joint FL_thigh_rotor_joint
- removed joint FR_calf_rotor_joint
- removed joint FR_hip_rotor_joint
- removed joint FR_thigh_rotor_joint
- removed joint RL_calf_rotor_joint
- removed joint RL_hip_rotor_joint
- removed joint RL_thigh_rotor_joint
- removed joint RR_calf_rotor_joint
- removed joint RR_hip_rotor_joint
- removed joint RR_thigh_rotor_joint
- removed joint front_camera_joint
- joint FL_hip_joint: parent base -> base_link
- joint FR_hip_joint: parent base -> base_link
- joint Head_upper_joint: parent base -> base_link
- joint RL_hip_joint: parent base -> base_link
- joint RR_hip_joint: parent base -> base_link
- joint imu_joint: parent base -> base_link
- joint radar_joint: parent base -> base_link

File: src/robots/go2/go2_description/xacro/const.xacro (robot description, xacro)
@@ -32,19 +32,10 @@
     <xacro:property name="hip_offset_y" value="0.0465"/>
     <xacro:property name="hip_offset_z" value="0.0"/>
-    <xacro:property name="hip_rotor_offset_x" value="0.11215"/>
-    <xacro:property name="hip_rotor_offset_y" value="0.04675"/>
-    <xacro:property name="hip_rotor_offset_z" value="0.0"/>
     <xacro:property name="thigh_offset_x" value="0"/>
     <xacro:property name="thigh_offset_y" value="0.0955"/>
     <xacro:property name="thigh_offset_z" value="0.0"/>
-    <xacro:property name="thigh_rotor_offset_x" value="0.0"/>
-    <xacro:property name="thigh_rotor_offset_y" value="-0.00015"/>
-    <xacro:property name="thigh_rotor_offset_z" value="0.0"/>
     <xacro:property name="calf_offset_x" value="0.0"/>
     <xacro:property name="calf_offset_y" value="0.0"/>
     <xacro:property name="calf_offset_z" value="-0.213"/>
-    <xacro:property name="calf_rotor_offset_x" value="0.0"/>
-    <xacro:property name="calf_rotor_offset_y" value="-0.03235"/>
-    <xacro:property name="calf_rotor_offset_z" value="0.0"/>
     <!-- joint limits -->
     <xacro:property name="damping" value="0.0"/>
@@ -85,14 +76,4 @@
     <xacro:property name="hip_iyz" value="-1.42E-06"/>
     <xacro:property name="hip_izz" value="0.000596"/>
-    <xacro:property name="hip_rotor_mass" value="0.089"/>
-    <xacro:property name="hip_rotor_com_x" value="0.0"/>
-    <xacro:property name="hip_rotor_com_y" value="0.0"/>
-    <xacro:property name="hip_rotor_com_z" value="0.0"/>
-    <xacro:property name="hip_rotor_ixx" value="0.000111842"/>
-    <xacro:property name="hip_rotor_ixy" value="0.0"/>
-    <xacro:property name="hip_rotor_ixz" value="0.0"/>
-    <xacro:property name="hip_rotor_iyy" value="0.000059647"/>
-    <xacro:property name="hip_rotor_iyz" value="0.0"/>
-    <xacro:property name="hip_rotor_izz" value="0.000059647"/>
     <!-- thigh -->
     <xacro:property name="thigh_mass" value="1.152"/>
@@ -106,14 +87,4 @@
     <xacro:property name="thigh_iyz" value="0.000808"/>
     <xacro:property name="thigh_izz" value="0.00103"/>
-    <xacro:property name="thigh_rotor_mass" value="0.089"/>
-    <xacro:property name="thigh_rotor_com_x" value="0.0"/>
-    <xacro:property name="thigh_rotor_com_y" value="0.0"/>
-    <xacro:property name="thigh_rotor_com_z" value="0.0"/>
-    <xacro:property name="thigh_rotor_ixx" value="0.000059647"/>
-    <xacro:property name="thigh_rotor_ixy" value="0.0"/>
-    <xacro:property name="thigh_rotor_ixz" value="0.0"/>
-    <xacro:property name="thigh_rotor_iyy" value="0.000111842"/>
-    <xacro:property name="thigh_rotor_iyz" value="0.0"/>
-    <xacro:property name="thigh_rotor_izz" value="0.000059647"/>
     <!-- calf -->
     <xacro:property name="calf_mass" value="0.154"/>
@@ -127,14 +98,4 @@
     <xacro:property name="calf_iyz" value="8.28E-06"/>
     <xacro:property name="calf_izz" value="3.29E-05"/>
-    <xacro:property name="calf_rotor_mass" value="0.089"/>
-    <xacro:property name="calf_rotor_com_x" value="0.0"/>
-    <xacro:property name="calf_rotor_com_y" value="0.0"/>
-    <xacro:property name="calf_rotor_com_z" value="0.0"/>
-    <xacro:property name="calf_rotor_ixx" value="0.000059647"/>
-    <xacro:property name="calf_rotor_ixy" value="0.0"/>
-    <xacro:property name="calf_rotor_ixz" value="0.0"/>
-    <xacro:property name="calf_rotor_iyy" value="0.000111842"/>
-    <xacro:property name="calf_rotor_iyz" value="0.0"/>
-    <xacro:property name="calf_rotor_izz" value="0.000059647"/>
     <!-- foot -->
     <xacro:property name="foot_mass" value="0.06"/>

File: src/robots/go2/go2_description/xacro/leg.xacro (robot description, xacro)
@@ -26,20 +26,4 @@
                 <limit effort="${hip_torque_max}" velocity="${hip_velocity_max}" lower="${-hip_position_max}" upper="${-hip_position_min}"/>
             </xacro:if>
-        </joint>
-        <joint name="${name}_hip_rotor_joint" type="fixed">
-            <xacro:if value="${(mirror_dae == False) and (front_hind_dae == True)}">
-                <origin rpy="0 0 0" xyz="${hip_rotor_offset_x} ${-hip_rotor_offset_y} 0"/>
-            </xacro:if>
-            <xacro:if value="${(mirror_dae == True) and (front_hind_dae == True)}">
-                <origin rpy="0 0 0" xyz="${hip_rotor_offset_x} ${hip_rotor_offset_y} 0"/>
-            </xacro:if>
-            <xacro:if value="${(mirror_dae == False) and (front_hind_dae == False)}">
-                <origin rpy="0 0 0" xyz="${-hip_rotor_offset_x} ${-hip_rotor_offset_y} 0"/>
-            </xacro:if>
-            <xacro:if value="${(mirror_dae == True) and (front_hind_dae == False)}">
-                <origin rpy="0 0 0" xyz="${-hip_rotor_offset_x} ${hip_rotor_offset_y} 0"/>
-            </xacro:if>
-            <parent link="trunk"/>
-            <child link="${name}_hip_rotor"/>
         </joint>
         <link name="${name}_hip">
@@ -77,27 +61,4 @@
             </inertial>
         </link>
-        <link name="${name}_hip_rotor">
-            <visual>
-                <origin rpy="0 ${PI/2.0} 0" xyz="0 0 0"/>
-                <geometry>
-                    <cylinder length="0.02" radius="0.035"/>
-                </geometry>
-                <material name="green"/>
-            </visual>
-            <!-- <collision>
-                <origin rpy="0 ${PI/2.0} 0" xyz="0 0 0"/>
-                <geometry>
-                    <cylinder length="0.02" radius="0.035"/>
-                </geometry>
-            </collision> -->
-            <inertial>
-                <origin rpy="0 0 0" xyz="${hip_rotor_com_x} ${hip_rotor_com_y} ${hip_rotor_com_z}"/>
-                <mass value="${hip_rotor_mass}"/>
-                <inertia
-                    ixx="${hip_rotor_ixx}" ixy="${hip_rotor_ixy}" ixz="${hip_rotor_ixz}"
-                    iyy="${hip_rotor_iyy}" iyz="${hip_rotor_iyz}"
-                    izz="${hip_rotor_izz}"/>
-            </inertial>
-        </link>
         <joint name="${name}_thigh_joint" type="revolute">
             <origin rpy="0 0 0" xyz="0 ${thigh_offset*mirror} 0"/>
@@ -107,9 +68,4 @@
             <dynamics damping="${damping}" friction="${friction}"/>
             <limit effort="${thigh_torque_max}" velocity="${thigh_velocity_max}" lower="${thigh_position_min}" upper="${thigh_position_max}"/>
-        </joint>
-        <joint name="${name}_thigh_rotor_joint" type="fixed">
-            <origin rpy="0 0 0" xyz="${thigh_rotor_offset_x} ${thigh_rotor_offset_y*mirror} 0"/>
-            <parent link="${name}_hip"/>
-            <child link="${name}_thigh_rotor"/>
         </joint>
         <link name="${name}_thigh">
@@ -141,27 +97,4 @@
             </inertial>
         </link>
-        <link name="${name}_thigh_rotor">
-            <visual>
-                <origin rpy="${PI/2.0} 0 0" xyz="0 0 0"/>
-                <geometry>
-                    <cylinder length="0.02" radius="0.035"/>
-                </geometry>
-                <material name="green"/>
-            </visual>
-            <!-- <collision>
-                <origin rpy="${PI/2.0} 0 0" xyz="0 0 0"/>
-                <geometry>
-                    <cylinder length="0.02" radius="0.035"/>
-                </geometry>
-            </collision> -->
-            <inertial>
-                <origin rpy="0 0 0" xyz="${thigh_rotor_com_x} ${thigh_rotor_com_y} ${thigh_rotor_com_z}"/>
-                <mass value="${thigh_rotor_mass}"/>
-                <inertia
-                    ixx="${thigh_rotor_ixx}" ixy="${thigh_rotor_ixy}" ixz="${thigh_rotor_ixz}"
-                    iyy="${thigh_rotor_iyy}" iyz="${thigh_rotor_iyz}"
-                    izz="${thigh_rotor_izz}"/>
-            </inertial>
-        </link>
         <joint name="${name}_calf_joint" type="revolute">
             <origin rpy="0 0 0" xyz="0 0 ${-thigh_length}"/>
@@ -171,9 +104,4 @@
             <dynamics damping="${damping}" friction="${friction}"/>
             <limit effort="${calf_torque_max}" velocity="${calf_velocity_max}" lower="${calf_position_min}" upper="${calf_position_max}"/>
-        </joint>
-        <joint name="${name}_calf_rotor_joint" type="fixed">
-            <origin rpy="0 0 0" xyz="${calf_rotor_offset_x} ${calf_rotor_offset_y*mirror} 0"/>
-            <parent link="${name}_thigh"/>
-            <child link="${name}_calf_rotor"/>
         </joint>
         <link name="${name}_calf">
@@ -200,28 +128,5 @@
             </inertial>
         </link>
-        <link name="${name}_calf_rotor">
-            <visual>
-                <origin rpy="${PI/2.0} 0 0" xyz="0 0 0"/>
-                <geometry>
-                    <cylinder length="0.02" radius="0.035"/>
-                </geometry>
-                <material name="green"/>
-            </visual>
-            <!-- <collision>
-                <origin rpy="${PI/2.0} 0 0" xyz="0 0 0"/>
-                <geometry>
-                    <cylinder length="0.02" radius="0.035"/>
-                </geometry>
-            </collision> -->
-            <inertial>
-                <origin rpy="0 0 0" xyz="${calf_rotor_com_x} ${calf_rotor_com_y} ${calf_rotor_com_z}"/>
-                <mass value="${calf_rotor_mass}"/>
-                <inertia
-                    ixx="${calf_rotor_ixx}" ixy="${calf_rotor_ixy}" ixz="${calf_rotor_ixz}"
-                    iyy="${calf_rotor_iyy}" iyz="${calf_rotor_iyz}"
-                    izz="${calf_rotor_izz}"/>
-            </inertial>
-        </link>
-        <joint name="${name}_foot_fixed" type="fixed">
+        <joint name="${name}_foot_fixed" type="fixed">0
             <origin rpy="0 0 0" xyz="0 0 ${-(calf_length)}"/>
             <parent link="${name}_calf"/>

File: src/robots/go2/go2_description/xacro/robot.xacro (robot description, xacro)
@@ -81,11 +81,4 @@
         </collision>
     </link>
-    <joint name="front_camera_joint" type="fixed">
-        <parent link="trunk"/>
-        <child link="front_camera"/>
-        <origin rpy="0 0 0" xyz="0.32715 -0.00003 0.04297"/>
-    </joint>
-    <link name="front_camera">
-    </link>
     <!--
     <joint name="load_joint" type="fixed">
